File: AKS_HBridge.kicad_pcb (KiCad board)
At the start: 4 copper layers, 1 part, among them U1 DRV8262DDVR

Commit message: pcb layout planning
Parts:
- added C1: 1uF, Capacitor_SMD:C_0603_1608Metric, F.Cu at (100.5, 88.8)
- added C2: 0.1uF, Capacitor_SMD:C_0402_1005Metric, F.Cu at (100.0, 98.5)
- added C3: 1uF, Capacitor_SMD:C_0402_1005Metric, F.Cu at (100.0, 100.5)
- added C4: 0.1uF, Capacitor_SMD:C_0603_1608Metric, F.Cu at (100.5, 91.3)
- added C5: 0.01uF, Capacitor_SMD:C_0603_1608Metric, F.Cu at (100.5, 93.8)
- added C6: 470uF, Capacitor_THT:CP_Radial_D16.0mm_P7.50mm, F.Cu at (86.0, 96.3)
- added C7: 0.01uF, Capacitor_SMD:C_0603_1608Metric, F.Cu at (100.5, 96.3)
- added C8: 0.1uF, Capacitor_SMD:C_0402_1005Metric, F.Cu at (100.0, 102.5)
- added J1: MOTA, Connector_Wire:SolderWirePad_1x01_SMD_5x10mm, F.Cu at (97.8, 110.8)
- added J2: MOTB, Connector_Wire:SolderWirePad_1x01_SMD_5x10mm, F.Cu at (104.3, 110.8)
- added J3: Control, Connector_JST:JST_PH_B5B-PH-K_1x05_P2.00mm_Vertical, F.Cu at (83.5, 107.8)
- added NT1: STARGND, NetTie:NetTie-2_SMD_Pad2.0mm, F.Cu at (84.0, 113.1)
- added R1: 10k, Resistor_SMD:R_0402_1005Metric, F.Cu at (104.0, 88.5)
- added R2: 47k, Resistor_SMD:R_0402_1005Metric, F.Cu at (104.0, 90.5)
- added R3: 47k, Resistor_SMD:R_0402_1005Metric, F.Cu at (104.0, 92.5)
Connections:
- U1 pad 1: GND -> GNDS
- U1 pad 14: Net-(U1-OUT2-Pad14) -> Net-(J2-Pin_1)
- U1 pad 15: Net-(U1-OUT2-Pad14) -> Net-(J2-Pin_1)
- U1 pad 16: Net-(U1-OUT2-Pad14) -> Net-(J2-Pin_1)
- U1 pad 17: Net-(TP1-Pad1) -> Net-(J1-Pin_1)
- U1 pad 18: Net-(TP1-Pad1) -> Net-(J1-Pin_1)
- U1 pad 19: Net-(TP1-Pad1) -> Net-(J1-Pin_1)
- U1 pad 22: unconnected-(U1-VCP-Pad22) -> Net-(U1-VCP)
- U1 pad 23: unconnected-(U1-CPH-Pad23) -> Net-(U1-CPH)
- U1 pad 24: unconnected-(U1-CPL-Pad24) -> Net-(U1-CPL)
- U1 pad 25: unconnected-(U1-SLEEP_N-Pad25) -> /SLEEP_N
- U1 pad 26: unconnected-(U1-IN1-Pad26) -> /IN1
- U1 pad 27: unconnected-(U1-IN2-Pad27) -> /IN2
- U1 pad 30: unconnected-(U1-DECAY-Pad30) -> GNDS
- U1 pad 33: unconnected-(U1-VREF1_VREF-Pad33) -> Net-(U1-VREF1_VREF)
- U1 pad 34: unconnected-(U1-VREF2_VREF-Pad34) -> Net-(U1-VREF1_VREF)
- U1 pad 36: unconnected-(U1-IPROPI1_IPROPI-Pad36) -> GNDS
- U1 pad 37: unconnected-(U1-IPROPI2_IPROPI-Pad37) -> GNDS
- U1 pad 38: unconnected-(U1-MODE2-Pad38) -> VCC
- U1 pad 39: unconnected-(U1-MODE1-Pad39) -> VCC
- U1 pad 4: Net-(U1-OUT3-Pad4) -> Net-(J1-Pin_1)
- U1 pad 40: unconnected-(U1-OCPM-Pad40) -> VCC
- U1 pad 41: unconnected-(U1-FAULT_N-Pad41) -> /FAULT_N
- U1 pad 42: unconnected-(U1-VCC-Pad42) -> VCC
- U1 pad 43: unconnected-(U1-DVDD-Pad43) -> VCC
- U1 pad 44: GND -> GNDS
- U1 pad 5: Net-(U1-OUT3-Pad4) -> Net-(J1-Pin_1)
- U1 pad 6: Net-(U1-OUT3-Pad4) -> Net-(J1-Pin_1)
- U1 pad 7: Net-(U1-OUT4-Pad7) -> Net-(J2-Pin_1)
- U1 pad 8: Net-(U1-OUT4-Pad7) -> Net-(J2-Pin_1)
- U1 pad 9: Net-(U1-OUT4-Pad7) -> Net-(J2-Pin_1)

Commit message: more layout and brought in refernce design
Parts:
- added J4: BATT+, Connector_Wire:SolderWirePad_1x01_SMD_5x10mm, F.Cu at (98.3, 124.9)
- added J5: BATT-, Connector_Wire:SolderWirePad_1x01_SMD_5x10mm, F.Cu at (105.8, 124.2)
- C5: moved to B.Cu
- moved C4 59.0 mm to (155.9, 111.6), turned to 90 degrees
- moved C1 49.7 mm to (144.4, 112.0), turned to -90 degrees
- moved C5 44.9 mm to (144.1, 104.6), turned to 90 degrees
